File: _autosave-JosEffigy-All-Keyboard-Mixbox.kicad_sch (KiCad schematic)
At the start: 33 parts, among them U1 Pico

Commit message: Release 1.0
Parts:
- MX8: footprint Button_Switch_Keyboard:SW_Cherry_MX_2.00u_Plate -> PCM_Switch_Keyboard_Hotswap_Kailh:SW_Hotswap_Kailh_MX_Plated_2.00u
Changed lines of the file:
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@@
       (effects (font (size 0.508 0.508)))
     )
-    (property "Footprint" "Button_Switch_Keyboard:SW_Cherry_MX_2.00u_Plate" (at 160.655 113.665 0)
+    (property "Footprint" "PCM_Switch_Keyboard_Hotswap_Kailh:SW_Hotswap_Kailh_MX_Plated_2.00u" (at 160.655 113.665 0)
       (effects (font (size 1.524 1.524)) hide)
     )
